File: Pi_CPU_002.brd (EAGLE design)
At the start: 49.2 x 85.1 mm, 34 parts, among them IC1 ULN2803, IC2 PCF8574TS, IC3 LD117AS50TR, X1 AK550/2

Commit message: Version 002
Routing:
- net IMR3: track 19.1 -> 18.4 mm
- net IMR2: track 16.8 -> 16.1 mm
- net GND: vias 10 -> 13
Changed lines of the file:
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@@
 <grid distance="0.05" unitdist="inch" unit="mm" style="lines" multiple="1" display="no" altdistance="0.1" altunitdist="mm" altunit="mm"/>
 <layers>
-<layer number="1" name="Top" color="4" fill="1" visible="no" active="yes"/>
+<layer number="1" name="Top" color="4" fill="1" visible="yes" active="yes"/>
 <layer number="16" name="Bottom" color="1" fill="1" visible="yes" active="yes"/>
 <layer number="17" name="Pads" color="2" fill="1" visible="yes" active="yes"/>
@@
 <layer number="220" name="220bmp" color="21" fill="1" visible="no" active="no"/>
 <layer number="221" name="221bmp" color="22" fill="1" visible="no" active="no"/>
-<layer number="222" name="222bmp" color="23" fill="1" visible="no" active="no"/>
 <layer number="223" name="223bmp" color="24" fill="1" visible="no" active="no"/>
 <layer number="224" name="224bmp" color="25" fill="1" visible="no" active="no"/>
@@
 <contactref element="SV2" pad="4"/>
 <contactref element="C3" pad="1"/>
+<via x="24.09" y="61.46" extent="1-16" drill="0.6"/>
+<via x="21.64" y="61.5" extent="1-16" drill="0.6"/>
+<via x="31.71" y="61.46" extent="1-16" drill="0.6"/>
 </signal>
 <signal name="A0">
@@
 <contactref element="IC1" pad="3"/>
 <contactref element="IC2" pad="17"/>
-<wire x1="23.79" y1="57.46" x2="23.79" y2="60.03" width="0.3048" layer="1"/>
-<wire x1="23.79" y1="60.03" x2="22.86" y2="60.96" width="0.3048" layer="1"/>
-<wire x1="22.86" y1="60.96" x2="22.86" y2="69.35" width="0.3048" layer="1"/>
+<wire x1="23.79" y1="57.46" x2="23.79" y2="58.76" width="0.3048" layer="1"/>
+<wire x1="23.79" y1="58.76" x2="22.86" y2="59.69" width="0.3048" layer="1"/>
+<wire x1="22.86" y1="59.69" x2="22.86" y2="69.35" width="0.3048" layer="1"/>
 <contactref element="RN1" pad="4"/>
 <wire x1="22.86" y1="69.35" x2="22.86" y2="66.65" width="0.6096" layer="16"/>
@@
 <contactref element="IC1" pad="5"/>
 <contactref element="IC2" pad="14"/>
-<wire x1="25.74" y1="57.46" x2="25.74" y2="60.03" width="0.3048" layer="1"/>
-<wire x1="25.74" y1="60.03" x2="27.94" y2="62.23" width="0.3048" layer="1"/>
-<wire x1="27.94" y1="62.23" x2="27.94" y2="69.35" width="0.3048" layer="1"/>
+<wire x1="25.74" y1="57.46" x2="25.74" y2="58.76" width="0.3048" layer="1"/>
+<wire x1="25.74" y1="58.76" x2="27.94" y2="60.96" width="0.3048" layer="1"/>
+<wire x1="27.94" y1="60.96" x2="27.94" y2="69.35" width="0.3048" layer="1"/>
 <contactref element="RN1" pad="6"/>
 <wire x1="27.94" y1="69.35" x2="27.94" y2="66.65" width="0.6096" layer="16"/>
@@
 <contactref element="IC1" pad="6"/>
 <contactref element="IC2" pad="12"/>
-<wire x1="27.94" y1="60.96" x2="29.21" y2="60.96" width="0.3048" layer="1"/>
+<wire x1="27.04" y1="57.46" x2="27.04" y2="58.79" width="0.3048" layer="1"/>
+<wire x1="27.04" y1="58.79" x2="29.21" y2="60.96" width="0.3048" layer="1"/>
 <wire x1="29.21" y1="60.96" x2="30.48" y2="62.23" width="0.3048" layer="1"/>
 <wire x1="30.48" y1="62.23" x2="30.48" y2="69.35" width="0.3048" layer="1"/>
-<wire x1="27.04" y1="57.46" x2="27.04" y2="60.06" width="0.3048" layer="1"/>
-<wire x1="27.04" y1="60.06" x2="27.94" y2="60.96" width="0.3048" layer="1"/>
 <contactref element="RN1" pad="7"/>
 <wire x1="30.48" y1="69.35" x2="30.48" y2="66.65" width="0.6096" layer="16"/>
@@
 <contactref element="IC1" pad="7"/>
 <contactref element="IC2" pad="11"/>
-<wire x1="27.69" y1="57.46" x2="27.69" y2="59.44" width="0.3048" layer="1"/>
-<wire x1="27.69" y1="59.44" x2="27.94" y2="59.69" width="0.3048" layer="1"/>
-<wire x1="27.94" y1="59.69" x2="31.75" y2="59.69" width="0.3048" layer="1"/>
+<wire x1="27.69" y1="57.46" x2="27.69" y2="58.17" width="0.3048" layer="1"/>
+<wire x1="27.69" y1="58.17" x2="29.21" y2="59.69" width="0.3048" layer="1"/>
+<wire x1="29.21" y1="59.69" x2="31.75" y2="59.69" width="0.3048" layer="1"/>
 <wire x1="31.75" y1="59.69" x2="33.02" y2="60.96" width="0.3048" layer="1"/>
 <wire x1="33.02" y1="60.96" x2="33.02" y2="69.35" width="0.3048" layer="1"/>
